Commit message: Sliding mode control on arm implemented

File: dynamics/arm.urdf (robot description, URDF)
Before this commit: robot arm_with_load, 4 links, 3 joints
Links:
- link load: mass 1 -> None
- link lower_link: geometry visual cylinder length=1.1 radius=.05
Joints:
- joint hold: origin xyz=0 0 -1.15 -> xyz=0 0 -0.65
